File: PCB/SmartPartsIONBoard.sch (KiCad schematic (older format))
At the start: 31 parts, among them J1 Conn_01x04, P1 TC2050-IDC, Q1 FDN337N, SW1 SW_Push, U1 MIC5205-2.5YM5, U2 MAX313CPE, U4 Logo-c, U5 ATmega328P-MU, Y2 Crystal

Commit message: Eye And Oled Display
Parts:
- added Brd1: SSD1306, ssd1306:128x64OLED, symbol SSD1306:SSD1306
- added D4: LED_Small, LED_THT:LED_D3.0mm_Horizontal_O1.27mm_Z2.0mm_IRBlack, symbol Device:LED_Small
- added J2: Conn_01x04, Ae_Logo:jst_4_smd, symbol Connector_Generic:Conn_01x04
- added Q2: Q_Photo_NPN, LED_THT:LED_D3.0mm_Horizontal_O1.27mm_Z2.0mm_Clear, symbol Device:Q_Photo_NPN
- added R8: 100R, Resistor_SMD:R_0603_1608Metric, symbol Device:R_US
- added R9: 10K, Resistor_SMD:R_0603_1608Metric, symbol Device:R_US
Connections:
- wire segments 76 -> 97
Other:
- moved on the sheet: D2, J1, L1, Q1, R1, R2, R3, R4, R6, SW1, U2A

Commit message: fix
Parts:
- removed C6, C7: C, Capacitor_SMD:C_1206_3216Metric, symbol Device:C
- removed P1: TC2050-IDC, Tag-Connect:TC2050-NL_SMALL, symbol Tag-Connect:TC2050-IDC
- removed Y2: Crystal, Crystal:Crystal_SMD_TXC_7A-2Pin_5x3.2mm, symbol Device:Crystal
- added R10, R11: R_Small_US, Resistor_SMD:R_0603_1608Metric, symbol Device:R_Small_US
- added SW2, SW3: SW_Push, Button_Switch_SMD:SW_Push_SPST_NO_Alps_SKRK, symbol Switch:SW_Push
Connections:
- wire segments 97 -> 93
- no-connect marks 2 -> 4
Other:
- moved on the sheet: R6, SW1
Changed lines of the file:
@@
 A1
 Wire Wire Line
-	6700 5100 6700 5500
+	5500 3775 5500 4175
 $Comp
 L Device:R_Small_US R6
 U 1 1 5D733949
-P 6700 5650
-F 0 "R6" H 6768 5696 50  0000 L CNN
-F 1 "R_Small_US" H 6768 5605 50  0000 L CNN
-F 2 "Resistor_SMD:R_0603_1608Metric" H 6700 5650 50  0001 C CNN
-F 3 "~" H 6700 5650 50  0001 C CNN
-	1    6700 5650
+P 5500 4325
+F 0 "R6" H 5568 4371 50  0000 L CNN
+F 1 "R_Small_US" H 5568 4280 50  0000 L CNN
+F 2 "Resistor_SMD:R_0603_1608Metric" H 5500 4325 50  0001 C CNN
+F 3 "~" H 5500 4325 50  0001 C CNN
+	1    5500 4325
 	1    0    0    -1
 $EndComp
@@
 L power:GND #PWR0110
 U 1 1 5D733950
-P 6700 5750
-F 0 "#PWR0110" H 6700 5500 50  0001 C CNN
-F 1 "GND" H 6705 5577 50  0000 C CNN
-F 2 "" H 6700 5750 50  0001 C CNN
-F 3 "" H 6700 5750 50  0001 C CNN
-	1    6700 5750
-	1    0    0    -1
-$EndComp
-Text GLabel 6700 5100 0    50   Input ~ 0
+P 5500 4425
+F 0 "#PWR0110" H 5500 4175 50  0001 C CNN
+F 1 "GND" H 5505 4252 50  0000 C CNN
+F 2 "" H 5500 4425 50  0001 C CNN
+F 3 "" H 5500 4425 50  0001 C CNN
+	1    5500 4425
+	1    0    0    -1
+$EndComp
+Text GLabel 5500 3775 0    50   Input ~ 0
 D4
 $Comp
 L Switch:SW_Push SW1
 U 1 1 5D73518D
-P 6900 5500
-F 0 "SW1" H 6900 5785 50  0000 C CNN
-F 1 "SW_Push" H 6900 5694 50  0000 C CNN
-F 2 "Button_Switch_SMD:SW_Push_SPST_NO_Alps_SKRK" H 6900 5700 50  0001 C CNN
-F 3 "~" H 6900 5700 50  0001 C CNN
-	1    6900 5500
-	1    0    0    -1
-$EndComp
-Connection ~ 6700 5500
-Wire Wire Line
-	6700 5500 6700 5550
+P 5700 4175
+F 0 "SW1" H 5700 4460 50  0000 C CNN
+F 1 "SW_Push" H 5700 4369 50  0000 C CNN
+F 2 "Button_Switch_SMD:SW_Push_SPST_NO_Alps_SKRK" H 5700 4375 50  0001 C CNN
+F 3 "~" H 5700 4375 50  0001 C CNN
+	1    5700 4175
+	1    0    0    -1
+$EndComp
+Connection ~ 5500 4175
+Wire Wire Line
+	5500 4175 5500 4225
 $Comp
 L power:VCC #PWR0111
 U 1 1 5D7459D1
-P 7250 5500
-F 0 "#PWR0111" H 7250 5350 50  0001 C CNN
-F 1 "VCC" H 7267 5673 50  0000 C CNN
-F 2 "" H 7250 5500 50  0001 C CNN
-F 3 "" H 7250 5500 50  0001 C CNN
-	1    7250 5500
+P 6050 4175
+F 0 "#PWR0111" H 6050 4025 50  0001 C CNN
+F 1 "VCC" H 6067 4348 50  0000 C CNN
+F 2 "" H 6050 4175 50  0001 C CNN
+F 3 "" H 6050 4175 50  0001 C CNN
+	1    6050 4175
 	0    1    1    0
 $EndComp
 Wire Wire Line
-	7100 5500 7250 5500
+	5900 4175 6050 4175
 $Comp
 L power:VCC #PWR0112
@@
 Text GLabel 8900 1750 2    50   Input ~ 0
 SCK
-Wire Wire Line
-	8800 2100 8500 2100
 Text GLabel 8500 1500 2    50   Input ~ 0
 D8
-Connection ~ 9100 2250
-Wire Wire Line
-	9600 2100 9400 2100
 $Comp
 L power:GND #PWR0108
@@
 	1    0    0    -1
 $EndComp
-Wire Wire Line
-	9600 2100 9600 2000
 Text GLabel 7300 1700 0    50   Input ~ 0
 A6
@@
 $EndComp
 Wire Wire Line
-	9400 2250 9400 2100
-Wire Wire Line
 	6900 1500 7300 1500
 Wire Wire Line
@@
 Text GLabel 8500 3600 2    50   Input ~ 0
 D4
-Wire Wire Line
-	8800 2250 9100 2250
 Text GLabel 8500 2800 2    50   Input ~ 0
 A4
@@
 $EndComp
 Wire Wire Line
-	8800 1950 8800 2100
-Connection ~ 9400 2100
-Wire Wire Line
 	8000 1200 7950 1200
 Wire Wire Line
@@
 Wire Wire Line
 	9050 3000 9050 3150
-Connection ~ 9100 1950
 Wire Wire Line
 	8750 2000 8500 2000
-Wire Wire Line
-	9400 2100 9400 1950
-Wire Wire Line
-	8800 2200 8800 2250
-Wire Wire Line
-	8500 2200 8800 2200
 $Comp
 L Device:C C9
@@
 $EndComp
 Wire Wire Line
-	8800 1950 9100 1950
-Wire Wire Line
 	9050 3000 8500 3000
 Text GLabel 8500 3700 2    50   Input ~ 0
@@
 Wire Wire Line
 	7950 1200 7950 900
-$Comp
-L Device:Crystal Y2
-U 1 1 5D707AC4
-P 9100 2100
-F 0 "Y2" V 9054 2231 50  0000 L CNN
-F 1 "Crystal" V 9145 2231 50  0000 L CNN
-F 2 "Crystal:Crystal_SMD_TXC_7A-2Pin_5x3.2mm" H 9100 2100 50  0001 C CNN
-F 3 "~" H 9100 2100 50  0001 C CNN
-	1    9100 2100
-	0    -1   -1   0
-$EndComp
-$Comp
-L power:GND #PWR0109
-U 1 1 5C4146B1
-P 9600 2000
-F 0 "#PWR0109" H 9600 1750 50  0001 C CNN
-F 1 "GND" H 9605 1827 50  0000 C CNN
-F 2 "" H 9600 2000 50  0001 C CNN
-F 3 "" H 9600 2000 50  0001 C CNN
-	1    9600 2000
-	-1   0    0    1
-$EndComp
 $Comp
 L MCU_Microchip_ATmega:ATmega328P-MU U5
@@
 NoConn ~ 4300 1600
 NoConn ~ 4550 1950
-$Comp
-L Device:C C6
-U 1 1 5D70FB57
-P 9250 2250
-F 0 "C6" V 8998 2250 50  0000 C CNN
-F 1 "C" V 9089 2250 50  0000 C CNN
-F 2 "Capacitor_SMD:C_1206_3216Metric" H 9288 2100 50  0001 C CNN
-F 3 "~" H 9250 2250 50  0001 C CNN
-	1    9250 2250
-	0    -1   -1   0
-$EndComp
-$Comp
-L Device:C C7
-U 1 1 5D70E7FC
-P 9250 1950
-F 0 "C7" V 8998 1950 50  0000 C CNN
-F 1 "C" V 9089 1950 50  0000 C CNN
-F 2 "Capacitor_SMD:C_1206_3216Metric" H 9288 1800 50  0001 C CNN
-F 3 "~" H 9250 1950 50  0001 C CNN
-	1    9250 1950
-	0    -1   -1   0
-$EndComp
-Text GLabel 4600 3350 0    50   Input ~ 0
-DTR2
-Text GLabel 4600 3050 0    50   Input ~ 0
-SCK
-Text GLabel 4600 3150 0    50   Input ~ 0
-MISO
-Text GLabel 4600 3250 0    50   Input ~ 0
-MOSI
-Text GLabel 5100 3150 2    50   Input ~ 0
-TXO
-Text GLabel 5100 3250 2    50   Input ~ 0
-DTR
-Text GLabel 4600 2950 0    50   Input ~ 0
-RESET
-Text GLabel 5100 2950 2    50   Input ~ 0
-GND
-Text GLabel 5100 3350 2    50   Input ~ 0
-VCC
-Text GLabel 5100 3050 2    50   Input ~ 0
-RXI
-$Comp
-L Tag-Connect:TC2050-IDC P1
-U 1 1 5DDBC776
-P 4850 3150
-F 0 "P1" H 4850 3539 40  0000 C CNN
-F 1 "TC2050-IDC" H 4850 3465 40  0000 C CNN
-F 2 "Tag-Connect:TC2050-NL_SMALL" H 4850 3150 50  0001 C CNN
-F 3 "" H 4850 3150 50  0001 C CNN
-	1    4850 3150
-	1    0    0    -1
-$EndComp
 $Comp
 L Connector_Generic:Conn_01x04 J1
@@
 Wire Wire Line
 	10175 4175 10375 4175
+Wire Wire Line
+	4350 3800 4350 4200
+$Comp
+L Device:R_Small_US R11
+U 1 1 5F3BC8B1
+P 4350 4350
+F 0 "R11" H 4418 4396 50  0000 L CNN
+F 1 "R_Small_US" H 4418 4305 50  0000 L CNN
+F 2 "Resistor_SMD:R_0603_1608Metric" H 4350 4350 50  0001 C CNN
+F 3 "~" H 4350 4350 50  0001 C CNN
+	1    4350 4350
+	1    0    0    -1
+$EndComp
+$Comp
+L power:GND #PWR0109
+U 1 1 5F3BC8B7
+P 4350 4450
+F 0 "#PWR0109" H 4350 4200 50  0001 C CNN
+F 1 "GND" H 4355 4277 50  0000 C CNN
+F 2 "" H 4350 4450 50  0001 C CNN
+F 3 "" H 4350 4450 50  0001 C CNN
+	1    4350 4450
+	1    0    0    -1
+$EndComp
+Text GLabel 4350 3800 0    50   Input ~ 0
+D4
+$Comp
+L Switch:SW_Push SW3
+U 1 1 5F3BC8BE
+P 4550 4200
+F 0 "SW3" H 4550 4485 50  0000 C CNN
+F 1 "SW_Push" H 4550 4394 50  0000 C CNN
+F 2 "Button_Switch_SMD:SW_Push_SPST_NO_Alps_SKRK" H 4550 4400 50  0001 C CNN
+F 3 "~" H 4550 4400 50  0001 C CNN
+	1    4550 4200
+	1    0    0    -1
+$EndComp
+Connection ~ 4350 4200
+Wire Wire Line
+	4350 4200 4350 4250
+$Comp
+L power:VCC #PWR0125
+U 1 1 5F3BC8C6
+P 4900 4200
+F 0 "#PWR0125" H 4900 4050 50  0001 C CNN
+F 1 "VCC" H 4917 4373 50  0000 C CNN
+F 2 "" H 4900 4200 50  0001 C CNN
+F 3 "" H 4900 4200 50  0001 C CNN
+	1    4900 4200
+	0    1    1    0
+$EndComp
+Wire Wire Line
+	4750 4200 4900 4200
+Wire Wire Line
+	3275 3800 3275 4200
+$Comp
+L Device:R_Small_US R10
+U 1 1 5F3C0D57
+P 3275 4350
+F 0 "R10" H 3343 4396 50  0000 L CNN
+F 1 "R_Small_US" H 3343 4305 50  0000 L CNN
+F 2 "Resistor_SMD:R_0603_1608Metric" H 3275 4350 50  0001 C CNN
+F 3 "~" H 3275 4350 50  0001 C CNN
+	1    3275 4350
+	1    0    0    -1
+$EndComp
+$Comp
+L power:GND #PWR0126
+U 1 1 5F3C0D5D
+P 3275 4450
+F 0 "#PWR0126" H 3275 4200 50  0001 C CNN
+F 1 "GND" H 3280 4277 50  0000 C CNN
+F 2 "" H 3275 4450 50  0001 C CNN
+F 3 "" H 3275 4450 50  0001 C CNN
+	1    3275 4450
+	1    0    0    -1
+$EndComp
+Text GLabel 3275 3800 0    50   Input ~ 0
+D4
+$Comp
+L Switch:SW_Push SW2
+U 1 1 5F3C0D64
+P 3475 4200
+F 0 "SW2" H 3475 4485 50  0000 C CNN
+F 1 "SW_Push" H 3475 4394 50  0000 C CNN
+F 2 "Button_Switch_SMD:SW_Push_SPST_NO_Alps_SKRK" H 3475 4400 50  0001 C CNN
+F 3 "~" H 3475 4400 50  0001 C CNN
+	1    3475 4200
+	1    0    0    -1
+$EndComp
+Connection ~ 3275 4200
+Wire Wire Line
+	3275 4200 3275 4250
+$Comp
+L power:VCC #PWR0128
+U 1 1 5F3C0D6C
+P 3825 4200
+F 0 "#PWR0128" H 3825 4050 50  0001 C CNN
+F 1 "VCC" H 3842 4373 50  0000 C CNN
+F 2 "" H 3825 4200 50  0001 C CNN
+F 3 "" H 3825 4200 50  0001 C CNN
+	1    3825 4200
+	0    1    1    0
+$EndComp
+Wire Wire Line
+	3675 4200 3825 4200
+NoConn ~ 8500 2100
+NoConn ~ 8500 2200
 $EndSCHEMATC
